File: F051_ESC-4in1-V2.kicad_pcb (KiCad board)
At the start: 4 copper layers, 46 x 55.8 mm, 223 parts, among them J1 Conn_01x02, J10 Conn_01x03, J11 Conn_01x03, J2 Conn_01x10, J3 Conn_01x04, J4 Conn_01x04, J5 Conn_01x04, J6 Conn_01x03, J7 Conn_01x04, J8 Conn_01x03, J9 Conn_01x10, Q1 TPH1R204PB, Q10 TPH1R204PB, Q11 TPH1R204PB, Q12 TPH1R204PB, Q13 TPH1R204PB, Q14 TPH1R204PB, Q15 TPH1R204PB, Q16 TPH1R204PB, Q17 TPH1R204PB, Q18 TPH1R204PB, Q19 TPH1R204PB, Q2 TPH1R204PB, Q20 TPH1R204PB, Q21 TPH1R204PB, Q22 TPH1R204PB, Q23 TPH1R204PB, Q24 TPH1R204PB, Q3 TPH1R204PB, Q4 TPH1R204PB, Q5 TPH1R204PB, Q6 TPH1R204PB, Q7 TPH1R204PB, Q8 TPH1R204PB, Q9 TPH1R204PB, U1 FD6288Q, U10 FD6288Q, U11 FD6288Q, U12 STM32F051K6Ux, U13 L78L12_SOT89, U14 MP4560_QFN10, U2 STM32F051K6Ux, U3 L78L12_SOT89, U4 LP2985-3.3, U5 INA139, U6 STM32F051K6Ux, U7 OPA340NA, U8 FD6288Q, U9 STM32F051K6Ux

Commit message: Added stuff
Parts:
- removed G***: LOGO, Footprints:DTOM_L
- added U15: DTOM, Footprints:DTOM_L, F.Cu at (140.5, 88.8)
- J2: footprint Connector_JST:JST_SHL_SM10B-SHLS-TF_1x10-1MP_P1.00mm_Horizontal -> Connector_JST:JST_SH_SM10B-SRSS-TB_1x10-1MP_P1.00mm_Horizontal
- moved J7 0.55 mm to (140.9, 76.8)
- moved J2 0.23 mm to (140.0, 65.5)
- moved C1 0.22 mm to (142.2, 91.7)
- moved R25 0.05 mm to (141.5, 88.7)
Routing:
- net +3V3: track 94.9 -> 99.8 mm
- net +12V_1: track 28.4 -> 31.9 mm
- net /MCU_4/USART1_RX: track 9.92 -> 12.9 mm
- net /MCU 3/PhaseB: track 23.0 -> 25.7 mm
- net VCC_Shunt: track 12.6 -> 14.5 mm, vias 133 -> 135
- net /MCU_4/USART1_TX: track 11.6 -> 13.2 mm
- net Net-(Q18-Pad4): track 9.90 -> 8.71 mm
- net /MCU_1/PhaseC: track 34.7 -> 35.7 mm
- net /Curent Sense/CURR: track 45.3 -> 46.3 mm
- net /MCU_1/SenseCOM: track 15.9 -> 15.0 mm
- net /MCU_1/PhaseA: track 33.3 -> 32.4 mm
- net +12V_2: track 35.0 -> 35.7 mm
- net /MOSFET_Driver_4/LO2: track 11.1 -> 10.5 mm
- net Net-(Q15-Pad4): track 9.76 -> 10.3 mm
- net /PWM_1: track 43.0 -> 43.6 mm
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Other:
- outline, holes or cut-outs redrawn

Commit message: Added stuff
Other:
- board text added: "1. Signal 2. GND 3. Signal 30-40 mil gap 4. Signal 5. PWR 6. Signal"
Changed lines of the file:
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@@
   (general
     (thickness 1.6)
-    (drawings 63)
+    (drawings 65)
     (tracks 2158)
     (zones 0)
@@
     (39 F.Mask user hide)
     (41 Cmts.User user hide)
-    (44 Edge.Cuts user)
+    (44 Edge.Cuts user hide)
     (45 Margin user hide)
-    (46 B.CrtYd user hide)
-    (47 F.CrtYd user hide)
+    (46 B.CrtYd user)
+    (47 F.CrtYd user)
     (48 B.Fab user hide)
     (49 F.Fab user hide)
@@
       (net 33 "/MCU 3/PhaseC"))
   )
+  (gr_circle (center 155.25 73.26) (end 158.25 73.26) (layer Cmts.User) (width 0.15))
+  (gr_text "1. Signal\n2. GND\n3. Signal\n30-40 mil gap\n4. Signal\n5. PWR\n6. Signal" (at 172.3 74.73) (layer Cmts.User)
+    (effects (font (size 1 1) (thickness 0.15)))
+  )
   (gr_line (start 155.25 68.5) (end 158.25 68.5) (layer Edge.Cuts) (width 0.15))
